File: getting-started/getting-started.kicad_sch (KiCad schematic)
At the start: 10 parts, among them SW1 SW_Push, SW2 SW_Push, SW3 SW_Push

Commit message: Finished with my first porject
Parts:
- added D1: LED, symbol Device:LED
- added R4: 1k, symbol Device:R
- added U1: MAX30102, symbol Spo2_stuff:MAX30102_Module
- added U2: SSD1306, symbol Spo2_stuff:SSD1306
Connections:
- net +5V: now also U1.5 (VCC), U2.2 (VCC)
- net GND: now also D1.1 (K), U1.4 (GND), U2.1 (GND)
- net at A1.15 (D12): now also R4.1
- net at A1.23 (A4): now also U1.2 (SDA), U2.4 (SDA)
- net at A1.24 (A5): now also U1.3 (SCL), U2.3 (SCL)
- new net: D1.2 (A), R4.2
- no-connect marks 0 -> 21
